Commit message: deleted unnecessary pkgs

File: husky_description/urdf/husky.urdf.xacro (robot description, xacro)
@@ -32,5 +32,4 @@
   <xacro:property name="husky_rear_bumper_extend" value="$(optenv HUSKY_REAR_BUMPER_EXTEND 0)" />
   <xacro:arg name="robot_namespace" default="/" />
-  <xacro:arg name="urdf_extras" default="empty.urdf" />
   <!-- Included URDF/XACRO Files -->
   <xacro:include filename="$(find husky_description)/urdf/decorations.urdf.xacro" />
@@ -128,5 +127,5 @@
   <joint name="camera_joint" type="fixed">
     <axis xyz="0 1 0" />
-    <origin xyz=".2 0 0.4" rpy="0 0 0"/>
+    <origin xyz=".2 0 0.8" rpy="0 0 0"/>
     <parent link="base_link"/>
     <child link="camera"/>
@@ -235,11 +234,9 @@
   </gazebo>
   <xacro:include filename="$(find velodyne_description)/urdf/VLP-16.urdf.xacro"/>
-  <xacro:VLP-16 parent="base_link" name="vlp201" topic="/vlp_1/velodyne_points" hz="20" samples="1845" gpu="true">
+  <xacro:VLP-16 parent="base_link" name="vlp201" topic="/vlp_1/velodyne_points" hz="40" samples="180" gpu="false">
     <origin xyz="0 0 0.35" rpy="0 0 0" />
   </xacro:VLP-16>
-  <xacro:VLP-16 parent="base_link" name="vlp202" topic="/vlp_2/velodyne_points" hz="20" samples="1845" gpu="true">
+  <xacro:VLP-16 parent="base_link" name="vlp202" topic="/vlp_2/velodyne_points" hz="40" samples="180" gpu="false">
     <origin xyz="0 -0.15 0.3" rpy="-1.57 3.14 3.14" />
   </xacro:VLP-16>
-  <!-- Optional custom includes. -->
-  <xacro:include filename="$(arg urdf_extras)" />
 </robot>

Commit message: now it works but only in environment rich in obstacles

File: husky_description/urdf/husky.urdf.xacro (robot description, xacro)
@@ -98,5 +98,5 @@
   <link name="imu_link"/>
   <joint name="imu_joint" type="fixed">
-    <origin xyz="$(optenv HUSKY_IMU_XYZ 0.19 0 0.149)" rpy="$(optenv HUSKY_IMU_RPY 0 -1.5708 3.1416)" />
+    <origin xyz="0 0 0" rpy="0 0 0" />
     <parent link="base_link" />
     <child link="imu_link" />
